File: kicadProject/MuMo-v2-Node.kicad_sch (KiCad schematic)
At the start: 75 parts, among them Q1 PJC7400, SW1 Reset, U1 MCP73123T-22SI/MF, U2 LoRa-E5, U3 CP2102N-Axx-xQFN24, U4 eInk_Display_1.54"200x200px, U5 BME680, U6 TSL25911, U7 BR24G512FVT-5AE2, U8 BR24G512FVT-5AE2

Commit message: add 3d model for enclosure
Parts:
- CONN2: value B2B-XH-A (LF)(SN) -> B2B-XH-A(LF)(SN); MPN B2B-XH-A (LF)(SN) -> B2B-XH-A(LF)(SN); supplier1Name Farnell -> DigiKey; supplier1PartNumber 1516276 -> 455-2247-ND; supplier1PartURL https://be.farnell.com/jst-japan-solderless-terminals/b2b-x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 -> https://www.digikey.be/nl/products/detail/jst-sales-america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
